Commit message: effort

File: agx_tutorial_resources/agx_tutorial_resources_panda_moveit_config/config/panda.ros2_control.xacro (robot description, xacro)
@@ -1,5 +1,5 @@
 <?xml version="1.0"?>
 <robot xmlns:xacro="http://www.ros.org/wiki/xacro">
-    <xacro:macro name="panda_ros2_control" params="name initial_positions_file ros2_control_hardware_type">
+    <xacro:macro name="panda_ros2_control" params="name initial_positions_file ros2_control_hardware_type command_interface">
         <xacro:property name="initial_positions" value="${xacro.load_yaml(initial_positions_file)['initial_positions']}"/>
         <ros2_control name="${name}" type="system">
@@ -15,5 +15,5 @@
             </hardware>
             <joint name="panda_joint1">
-                <command_interface name="position"/>
+                <command_interface name="${command_interface}"/>
                 <state_interface name="position">
                   <param name="initial_value">${initial_positions['panda_joint1']}</param>
@@ -22,5 +22,5 @@
             </joint>
             <joint name="panda_joint2">
-                <command_interface name="position"/>
+                <command_interface name="${command_interface}"/>
                 <state_interface name="position">
                   <param name="initial_value">${initial_positions['panda_joint2']}</param>
@@ -29,5 +29,5 @@
             </joint>
             <joint name="panda_joint3">
-                <command_interface name="position"/>
+                <command_interface name="${command_interface}"/>
                 <state_interface name="position">
                   <param name="initial_value">${initial_positions['panda_joint3']}</param>
@@ -36,5 +36,5 @@
             </joint>
             <joint name="panda_joint4">
-                <command_interface name="position"/>
+                <command_interface name="${command_interface}"/>
                 <state_interface name="position">
                   <param name="initial_value">${initial_positions['panda_joint4']}</param>
@@ -43,5 +43,5 @@
             </joint>
             <joint name="panda_joint5">
-                <command_interface name="position"/>
+                <command_interface name="${command_interface}"/>
                 <state_interface name="position">
                   <param name="initial_value">${initial_positions['panda_joint5']}</param>
@@ -50,5 +50,5 @@
             </joint>
             <joint name="panda_joint6">
-                <command_interface name="position"/>
+                <command_interface name="${command_interface}"/>
                 <state_interface name="position">
                   <param name="initial_value">${initial_positions['panda_joint6']}</param>
@@ -57,5 +57,5 @@
             </joint>
             <joint name="panda_joint7">
-                <command_interface name="position"/>
+                <command_interface name="${command_interface}"/>
                 <state_interface name="position">
                   <param name="initial_value">${initial_positions['panda_joint7']}</param>

File: agx_tutorial_resources/agx_tutorial_resources_panda_moveit_config/config/panda.urdf.xacro (robot description, xacro)
@@ -8,5 +8,5 @@
     <xacro:include filename="panda.ros2_control.xacro" />
     <xacro:include filename="panda_hand.ros2_control.xacro" />
-    <xacro:panda_ros2_control name="PandaFakeSystem" initial_positions_file="$(arg initial_positions_file)" ros2_control_hardware_type="$(arg ros2_control_hardware_type)"/>
+    <xacro:panda_ros2_control name="PandaFakeSystem" initial_positions_file="$(arg initial_positions_file)" ros2_control_hardware_type="$(arg ros2_control_hardware_type)" command_interface="$(arg command_interface)"/>
     <xacro:panda_hand_ros2_control name="PandaHandFakeSystem" ros2_control_hardware_type="$(arg ros2_control_hardware_type)"/>
 </robot>
