Commit message: remove panda_finger_joint2 from ros2_control

File: agx_tutorial_resources/agx_tutorial_resources_panda_moveit_config/config/panda_hand.ros2_control.xacro (robot description, xacro)
@@ -20,13 +20,4 @@
                 <state_interface name="velocity"/>
             </joint>
-            <joint name="panda_finger_joint2">
-                <param name="mimic">panda_finger_joint1</param>
-                <param name="multiplier">1</param>
-                <command_interface name="position" />
-                <state_interface name="position">
-                  <param name="initial_value">0.0</param>
-                </state_interface>
-                <state_interface name="velocity"/>
-            </joint>
         </ros2_control>
     </xacro:macro>
