Commit message: panda link masses according to this
https://github.com/frankaemika/franka_ros/blob/develop/franka_description/robots/common/inertial.yaml

File: agx_tutorial_resources/agx_tutorial_resources_panda_description/urdf/panda.urdf (robot description, URDF)
Before this commit: robot panda, 13 links, 12 joints
Links:
- link panda_hand: mass 0.68 -> 0.73
- link panda_leftfinger: mass 0.01 -> 0.015
- link panda_link0: mass 3.06 -> 0.629769
- link panda_link1: mass 2.34 -> 4.970684
- link panda_link2: mass 2.36 -> 0.646926
- link panda_link3: mass 2.38 -> 3.228604
- link panda_link4: mass 2.43 -> 3.587895
- link panda_link5: mass 3.5 -> 1.225946
- link panda_link6: mass 1.47 -> 1.666555
- link panda_link7: mass 0.45 -> 7.35522e-01
- link panda_rightfinger: mass 0.01 -> 0.015

Commit message: remove link8 inertia

File: agx_tutorial_resources/agx_tutorial_resources_panda_description/urdf/panda.urdf (robot description, URDF)
Before this commit: robot panda, 13 links, 12 joints
Links:
- link panda_link8: mass 0.1 -> None
